File: eagle/808-Maraca.sch (EAGLE design)
At the start: 46 parts, among them IC1 TL071P, Q1 2N3904, Q2 2N3906, Q3 2N3906, Q4 2N3904, Q59 2N3904, Q60 2N3906

Commit message: cutout
Parts:
- added C10, C9: 10n, TR808clone:C-EU050-024X044
- C8: device TR808clone:C-EU050-024X044 -> TR808clone:C-EU025-025X050
- R14: device TR808clone:R-EU_0207/5V -> TR808clone:R-EU_0207/2V
Connections:
- net +12V: now also C10.1
- net -12V: now also C9.2
- net GND: now also C10.2, C9.1
Changed lines of the file:
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@@
 <part name="IC1" library="linear" deviceset="TL071" device="P"/>
 <part name="R13" library="TR808clone" deviceset="R-EU_" device="0207/7" value="470K"/>
-<part name="C8" library="TR808clone" deviceset="C-EU" device="050-024X044" value="220p"/>
+<part name="C8" library="TR808clone" deviceset="C-EU" device="025-025X050" value="220p"/>
 <part name="P+5" library="supply1" deviceset="+12V" device=""/>
 <part name="P-3" library="supply1" deviceset="-12V" device=""/>
-<part name="R14" library="TR808clone" deviceset="R-EU_" device="0207/5V" value="47K"/>
+<part name="R14" library="TR808clone" deviceset="R-EU_" device="0207/2V" value="47K"/>
 <part name="V13" library="supply1" deviceset="GND" device=""/>
 <part name="WHITE_NOISE" library="erthenvar" deviceset="AUDIO-JACK" device=""/>
 <part name="V14" library="supply1" deviceset="GND" device=""/>
+<part name="P-4" library="supply1" deviceset="-12V" device=""/>
+<part name="P+6" library="supply1" deviceset="+12V" device=""/>
+<part name="C9" library="TR808clone" deviceset="C-EU" device="050-024X044" value="10n"/>
+<part name="C10" library="TR808clone" deviceset="C-EU" device="050-024X044" value="10n"/>
+<part name="V15" library="supply1" deviceset="GND" device=""/>
 </parts>
 <sheets>
@@
 <instance part="WHITE_NOISE" gate="G$1" x="187.96" y="50.8" rot="R180"/>
 <instance part="V14" gate="1" x="180.34" y="40.64" rot="MR0"/>
+<instance part="P-4" gate="1" x="147.32" y="104.14"/>
+<instance part="P+6" gate="1" x="147.32" y="134.62"/>
+<instance part="C9" gate="G$1" x="147.32" y="114.3" smashed="yes">
+<attribute name="NAME" x="150.241" y="112.776" size="1.778" layer="95" rot="R270"/>
+<attribute name="VALUE" x="142.621" y="115.316" size="1.778" layer="96" rot="R270"/>
+</instance>
+<instance part="C10" gate="G$1" x="147.32" y="127" smashed="yes">
+<attribute name="NAME" x="150.241" y="125.476" size="1.778" layer="95" rot="R270"/>
+<attribute name="VALUE" x="142.621" y="128.016" size="1.778" layer="96" rot="R270"/>
+</instance>
+<instance part="V15" gate="1" x="160.02" y="114.3"/>
 </instances>
 <busses>
@@
 <wire x1="180.34" y1="48.26" x2="180.34" y2="43.18" width="0.1524" layer="91"/>
 </segment>
+<segment>
+<pinref part="V15" gate="1" pin="GND"/>
+<wire x1="160.02" y1="116.84" x2="160.02" y2="119.38" width="0.1524" layer="91"/>
+<pinref part="C9" gate="G$1" pin="1"/>
+<pinref part="C10" gate="G$1" pin="2"/>
+<wire x1="147.32" y1="116.84" x2="147.32" y2="119.38" width="0.1524" layer="91"/>
+<wire x1="147.32" y1="119.38" x2="147.32" y2="121.92" width="0.1524" layer="91"/>
+<wire x1="160.02" y1="119.38" x2="147.32" y2="119.38" width="0.1524" layer="91"/>
+<junction x="147.32" y="119.38"/>
+</segment>
 </net>
 <net name="+12V" class="0">
@@
 <wire x1="210.82" y1="68.58" x2="210.82" y2="71.12" width="0.1524" layer="91"/>
 </segment>
+<segment>
+<pinref part="P+6" gate="1" pin="+12V"/>
+<pinref part="C10" gate="G$1" pin="1"/>
+<wire x1="147.32" y1="132.08" x2="147.32" y2="129.54" width="0.1524" layer="91"/>
+</segment>
 </net>
 <net name="-12V" class="0">
@@
 <wire x1="210.82" y1="88.9" x2="210.82" y2="86.36" width="0.1524" layer="91"/>
 </segment>
-</net>
+<segment>
+<pinref part="P-4" gate="1" pin="-12V"/>
+<pinref part="C9" gate="G$1" pin="2"/>
+<wire x1="147.32" y1="109.22" x2="147.32" y2="106.68" width="0.1524" layer="91"/>
+</segment>
+</net>
